File: hw/Carrier_Board/Carrier_Board.kicad_pcb (KiCad board)
At the start: 0 parts

Commit message: hw: initial schematic mostly done, pushing for reference
Parts:
- added C12: 0.1u, Capacitor_SMD:C_0603_1608Metric_Pad1.08x0.95mm_HandSolder, F.Cu at (101.6, 97.4)
- added C13: 4.7u, Capacitor_SMD:C_0805_2012Metric_Pad1.18x1.45mm_HandSolder, F.Cu at (106.2, 94.7)
- added C14: 0.1u, Capacitor_SMD:C_0603_1608Metric_Pad1.08x0.95mm_HandSolder, F.Cu at (101.6, 100.0)
- added C15: 0.1u, Capacitor_SMD:C_0603_1608Metric_Pad1.08x0.95mm_HandSolder, F.Cu at (101.6, 102.5)
- added C16: 0.1u, Capacitor_SMD:C_0603_1608Metric_Pad1.08x0.95mm_HandSolder, F.Cu at (101.6, 105.0)
- added C17: 4.7u, Capacitor_SMD:C_0805_2012Metric_Pad1.18x1.45mm_HandSolder, F.Cu at (106.2, 97.7)
- added C18: 0.1u, Capacitor_SMD:C_0603_1608Metric_Pad1.08x0.95mm_HandSolder, F.Cu at (101.6, 107.5)
- added C7: 0.1u, Capacitor_SMD:C_0603_1608Metric_Pad1.08x0.95mm_HandSolder, F.Cu at (101.6, 89.9)
- added C8: 0.1u, Capacitor_SMD:C_0603_1608Metric_Pad1.08x0.95mm_HandSolder, F.Cu at (101.6, 92.4)
- added C9: 0.1u, Capacitor_SMD:C_0603_1608Metric_Pad1.08x0.95mm_HandSolder, F.Cu at (101.6, 94.9)
- added D1: LED_Small_Filled, LED_SMD:LED_0603_1608Metric_Pad1.05x0.95mm_HandSolder, F.Cu at (71.6, 109.7)
- added D2: SS12, Diode_SMD:D_SMA, F.Cu at (107.8, 90.9)
- added D3: LED_Small_Filled, LED_SMD:LED_0603_1608Metric_Pad1.05x0.95mm_HandSolder, F.Cu at (71.6, 112.3)
- added D4: LED_Small_Filled, LED_SMD:LED_0603_1608Metric_Pad1.05x0.95mm_HandSolder, F.Cu at (71.6, 114.8)
- added D5: LED_Small_Filled, LED_SMD:LED_0603_1608Metric_Pad1.05x0.95mm_HandSolder, F.Cu at (71.6, 117.4)
- added F1: 500 mA, Fuse:Fuse_1206_3216Metric_Pad1.42x1.75mm_HandSolder, F.Cu at (68.5, 82.5)
- added R1: 10K, Resistor_SMD:R_0603_1608Metric_Pad0.98x0.95mm_HandSolder, F.Cu at (67.2, 109.6)
- added R2: 590, Resistor_SMD:R_0603_1608Metric_Pad0.98x0.95mm_HandSolder, F.Cu at (67.2, 112.1)
- added R3: 590, Resistor_SMD:R_0603_1608Metric_Pad0.98x0.95mm_HandSolder, F.Cu at (67.2, 114.7)
- added R4: 270, Resistor_SMD:R_0603_1608Metric_Pad0.98x0.95mm_HandSolder, F.Cu at (67.2, 117.2)
- added R5: 4.7K, Resistor_SMD:R_0603_1608Metric_Pad0.98x0.95mm_HandSolder, F.Cu at (101.6, 110.0)
- added R6: 4.7K, Resistor_SMD:R_0603_1608Metric_Pad0.98x0.95mm_HandSolder, F.Cu at (101.6, 112.5)
- added R7: 270, Resistor_SMD:R_0603_1608Metric_Pad0.98x0.95mm_HandSolder, F.Cu at (67.2, 119.7)
- added TP1: TestPoint, TestPoint:TestPoint_Keystone_5005-5009_Compact, F.Cu at (52.4, 110.9)
- added TP2: TestPoint, TestPoint:TestPoint_Keystone_5005-5009_Compact, F.Cu at (52.4, 116.0)
- added TP3: TestPoint, TestPoint:TestPoint_Keystone_5005-5009_Compact, F.Cu at (52.4, 121.0)
- added TP4: TestPoint, TestPoint:TestPoint_Keystone_5005-5009_Compact, F.Cu at (57.5, 110.9)
- added TP5: TestPoint, TestPoint:TestPoint_Keystone_5005-5009_Compact, F.Cu at (57.5, 116.0)
- added TP6: TestPoint, TestPoint:TestPoint_Keystone_5005-5009_Compact, F.Cu at (57.5, 121.0)
- added TP7: TestPoint, TestPoint:TestPoint_Keystone_5005-5009_Compact, F.Cu at (62.5, 110.9)
- added TP8: TestPoint, TestPoint:TestPoint_Keystone_5005-5009_Compact, F.Cu at (62.5, 116.0)
- added TP9: TestPoint, TestPoint:TestPoint_Keystone_5005-5009_Compact, F.Cu at (62.5, 121.0)
- added U4: HDC1080, Package_SON:Texas_PWSON-N6, F.Cu at (106.3, 101.6)
Other:
- copper layers 0 -> 2

Commit message: hw: initial layout done as well
Parts:
- removed C16: 0.1u, Capacitor_SMD:C_0603_1608Metric_Pad1.08x0.95mm_HandSolder
- added J1: Conn_01x05, Carrier_Board:JST_PA_S05B, F.Cu at (162.0, 78.0)
- added R8: 10K, Resistor_SMD:R_0603_1608Metric_Pad0.98x0.95mm_HandSolder, F.Cu at (150.0, 69.2)
- added R9: 10K, Resistor_SMD:R_0603_1608Metric_Pad0.98x0.95mm_HandSolder, F.Cu at (150.0, 77.5)
- added TP1: TestPoint, TestPoint:TestPoint_Keystone_5000-5004_Miniature, F.Cu at (105.0, 68.0)
- added TP2: TestPoint, TestPoint:TestPoint_Keystone_5000-5004_Miniature, F.Cu at (133.0, 79.5)
- added TP3: TestPoint, TestPoint:TestPoint_Keystone_5000-5004_Miniature, F.Cu at (105.0, 62.0)
- added TP4: TestPoint, TestPoint:TestPoint_Keystone_5000-5004_Miniature, F.Cu at (129.5, 79.5)
- added TP5: TestPoint, TestPoint:TestPoint_Keystone_5000-5004_Miniature, F.Cu at (105.0, 80.0)
- added TP6: TestPoint, TestPoint:TestPoint_Keystone_5000-5004_Miniature, F.Cu at (105.0, 73.0)
- added TP7: TestPoint, TestPoint:TestPoint_Keystone_5000-5004_Miniature, F.Cu at (105.0, 76.5)
- added U1: ~, Carrier_Board:Atom_S3-Lite, F.Cu at (121.0, 63.0)
- added U3: ~, Package_TO_SOT_SMD:SOT-23-6_Handsoldering, F.Cu at (145.0, 77.5)
- added U4: ~, Package_TO_SOT_SMD:SOT-23-6_Handsoldering, F.Cu at (145.0, 69.3)
- TP10: renamed from TP3; footprint TestPoint:TestPoint_Keystone_5005-5009_Compact -> TestPoint:TestPoint_Keystone_5000-5004_Miniature
- TP11: renamed from TP4; footprint TestPoint:TestPoint_Keystone_5005-5009_Compact -> TestPoint:TestPoint_Keystone_5000-5004_Miniature
- TP12: renamed from TP5; footprint TestPoint:TestPoint_Keystone_5005-5009_Compact -> TestPoint:TestPoint_Keystone_5000-5004_Miniature
- TP13: renamed from TP6; footprint TestPoint:TestPoint_Keystone_5005-5009_Compact -> TestPoint:TestPoint_Keystone_5000-5004_Miniature
- TP14: renamed from TP7; footprint TestPoint:TestPoint_Keystone_5005-5009_Compact -> TestPoint:TestPoint_Keystone_5000-5004_Miniature
- TP15: renamed from TP8; footprint TestPoint:TestPoint_Keystone_5005-5009_Compact -> TestPoint:TestPoint_Keystone_5000-5004_Miniature
- TP16: renamed from TP9; footprint TestPoint:TestPoint_Keystone_5005-5009_Compact -> TestPoint:TestPoint_Keystone_5000-5004_Miniature
- TP8: renamed from TP1; footprint TestPoint:TestPoint_Keystone_5005-5009_Compact -> TestPoint:TestPoint_Keystone_5000-5004_Miniature
- TP9: renamed from TP2; footprint TestPoint:TestPoint_Keystone_5005-5009_Compact -> TestPoint:TestPoint_Keystone_5000-5004_Miniature
- moved TP10 129.7 mm to (165.5, 57.5)
- moved TP11 119.0 mm to (162.0, 54.0)
- moved TP9 110.6 mm to (144.0, 54.0), turned to -90 degrees
- moved TP8 105.8 mm to (144.0, 58.0), turned to -90 degrees
- moved R3 103.4 mm to (153.0, 54.5)
- moved R6 101.2 mm to (156.5, 67.0)
- moved TP15 100.5 mm to (154.0, 74.5)
- moved TP16 100.3 mm to (154.0, 80.0)
- moved TP14 100.2 mm to (154.0, 70.0)
- moved TP12 100.0 mm to (152.5, 85.0)
- moved TP13 97.9 mm to (148.5, 85.0)
- moved D4 96.8 mm to (155.5, 64.0), turned to 90 degrees
- moved F1 95.6 mm to (162.0, 62.8), turned to -90 degrees
- moved D3 95.1 mm to (149.0, 54.5), turned to 180 degrees
- moved R2 84.4 mm to (137.5, 70.5)
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- renumbered C18 to C1, C17 to C2, C15 to C3, C13 to C4, C14 to C5, C12 to C6, C9 to C7, C7 to C9, D5 to D1, D4 to D2, D1 to D3, D3 to D4, D2 to D5, R7 to R1, R4 to R2, R2 to R3, R5 to R4, R6 to R5, R3 to R6, R1 to R7, U4 to U2
Routing:
- net /CN105_OE: track 0.00 -> 53.1 mm, vias 0 -> 2
- net GND: track 0.00 -> 47.7 mm, vias 0 -> 149
- net /STATUS_LED: track 0.00 -> 36.8 mm
- net /MODULE_SDA: track 0.00 -> 36.5 mm
- net /MODULE_SCL: track 0.00 -> 35.9 mm
- net 3V3: track 0.00 -> 26.3 mm
- net /CN105_TX_IN: track 0.00 -> 23.6 mm
- net /CN105_RX_OUT_3V3: track 0.00 -> 23.2 mm, vias 0 -> 1
- net 5V_CN105: track 0.00 -> 22.4 mm, vias 0 -> 3
- net 5V_MODULE: track 0.00 -> 20.2 mm
- net /CN105_RX_OUT: track 0.00 -> 18.6 mm
- net /CN105_TX_IN_3V3: track 0.00 -> 16.5 mm
- net /12V: track 0.00 -> 10.7 mm
- net Net-(D3-K): track 0.00 -> 2.21 mm
- net Net-(D1-K): track 0.00 -> 2.21 mm
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- added copper zone on F.Cu, net /CN105_5V_IN
- added copper zone on F.Cu, net 3V3
- added copper zone on F.Cu, net 5V_CN105
- added copper zone on B.Cu, net GND
Other:
- board outline added: 70 x 40 mm
- board text added: "12V"
- board text added: "3V3"
- board text added: "3V3 PWR"
- board text added: "5V"
- board text added: "< TX"
- board text added: "A"
- board text added: "CN105"
- board text added: "GND"
- board text added: "J1"
- board text added: "MITSUBISHI CN105 CONTROLLER"
- board text added: "MOD"
- board text added: "PWR"
- board text added: "REV"
- board text added: "REV A00 BOT"
- board text added: "REV A00 TOP"
- board text added: "RX >"
- board text added: "SCL"
- board text added: "SDA"
- board text added: "SN"

Commit message: hw: ready for initial quoting
Parts:
- added C5: 4.7u, Capacitor_SMD:C_0805_2012Metric_Pad1.18x1.45mm_HandSolder, F.Cu at (173.3, 92.0)
- J1: value Conn_01x05 -> JST PA-Series Header (Right-Angle)
- R3, R6: value 590 -> 620
- moved F1 34.0 mm to (178.0, 92.8)
- moved TP9 34.0 mm to (159.0, 84.5)
- moved R5 33.8 mm to (124.0, 112.6)
- moved C1 33.5 mm to (133.0, 112.7)
- moved C10 33.5 mm to (162.5, 102.3)
- moved C2 33.5 mm to (151.5, 107.0)
- moved C3 33.5 mm to (152.0, 87.0)
- moved C4 33.5 mm to (155.0, 87.0)
- moved C7 33.5 mm to (157.5, 104.5)
- moved C8 33.5 mm to (157.5, 102.3)
- moved C9 33.5 mm to (162.5, 104.5)
- moved D1 33.5 mm to (137.0, 109.5)
- moved D2 33.5 mm to (151.5, 97.5)
- moved D3 33.5 mm to (164.0, 84.5)
- moved D4 33.5 mm to (170.5, 94.0)
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- renumbered C9 to C10, C5 to C6, C6 to C7, C7 to C8, C8 to C9
Routing:
- net 3V3: track 26.3 -> 24.3 mm
- net GND: track 47.7 -> 46.5 mm, vias 149 -> 151
- net 5V_CN105: track 22.4 -> 23.2 mm, vias 3 -> 4
Other:
- rule pad_to_mask_clearance: 0 -> 0.05
- board text added: "0"
- board text added: "0 mm"
- board text added: "0.01 mm"
- board text added: "0.02"
- board text added: "0.035 mm"
- board text added: "0.1600 mm / 0.1800 mm"
- board text added: "0.3000 mm"
- board text added: "1"
- board text added: "1.51 mm"
- board text added: "1.6000 mm"
- board text added: "2"
- board text added: "3.3"
- board text added: "4.5"
- board text added: "70.0000 mm x 40.0000 mm"
- board text added: "<TX"
- board text added: "B.Cu"
- board text added: "B.Mask"
- board text added: "B.Paste"
- board text added: "B.Silkscreen"
- board text added: "BOARD CHARACTERISTICS"
- board text added: "Board Thickness:"
- board text added: "Board overall dimensions:"
- board text added: "Bottom Silk Screen"
- board text added: "Bottom Solder Mask"
- board text added: "Bottom Solder Paste"
- board text added: "Castellated pads:"
- board text added: "Color"
- board text added: "Copper Finish:"
- board text added: "Copper Layer Count:"
- board text added: "Dielectric 1"
- board text added: "ENIG"
- board text added: "Edge card connectors:"
- board text added: "Epsilon R"
- board text added: "F.Cu"
- board text added: "F.Mask"
- board text added: "F.Paste"
- board text added: "F.Silkscreen"
- board text added: "FR4"
- board text added: "Impedance Control:"
- board text added: "Layer Name"
- board text added: "Loss Tangent"
- board text added: "Material"
- board text added: "Min hole diameter:"
- board text added: "Min track/spacing:"
- board text added: "No"
- board text added: "Not specified"
- board text added: "Plated Board Edge:"
- board text added: "RX>"
- board text added: "Thickness (mm)"
- board text added: "Top Silk Screen"
- board text added: "Top Solder Mask"
- board text added: "Top Solder Paste"
- board text added: "Type"
- board text added: "copper"
- board text added: "core"
- board text removed: "< TX"
- board text removed: "RX >"

Commit message: hw: few little tweaks
Routing:
- net GND: vias 151 -> 152
Other:
- board text added: "ID"
- board text added: "MITSUBISHI CN105 INTERFACE MODULE"
- board text added: "REV A BOT"
- board text added: "REV A TOP"
- board text removed: "MITSUBISHI CN105 CONTROLLER"
- board text removed: "REV A00 BOT"
- board text removed: "REV A00 TOP"
Changed lines of the file:
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@@
 	(gr_poly
 		(pts
-			(xy 183 100.5) (xy 185 100.5) (xy 185 120) (xy 183 120)
+			(xy 183 98.5) (xy 185 98.5) (xy 185 120) (xy 183 120)
 		)
 		(stroke
@@
 	)
 	(gr_rect
-		(start 141 112)
-		(end 159 117)
+		(start 142 112.5)
+		(end 159 117.5)
 		(stroke
 			(width 0.1)
@@
 	)
 	(gr_rect
-		(start 166.61875 90.5)
-		(end 171.38125 93.5)
+		(start 136.5 95.38125)
+		(end 139.5 100.14375)
 		(stroke
 			(width 0.1)
@@
 	)
 	(gr_rect
-		(start 130.7625 113)
-		(end 149.2375 116)
+		(start 131.5 83.525)
+		(end 134.5 104)
 		(stroke
 			(width 0.1)
@@
 		(layer "F.Fab")
 	)
-	(gr_text "REV A00 TOP"
+	(gr_text "REV A TOP"
 		(at 184 89.5 270)
 		(layer "F.Cu")
@@
 		)
 	)
-	(gr_text "REV A00 BOT"
-		(at 184 99.3 270)
+	(gr_text "REV A BOT"
+		(at 184 98 270)
 		(layer "B.Cu")
 		(effects
@@
 	(gr_text "PWR"
 		(at 169 95.2 0)
-		(layer "F.SilkS")
+		(layer "F.SilkS" knockout)
 		(effects
 			(font
@@
 	(gr_text "3V3 PWR"
 		(at 139 115.5 90)
-		(layer "F.SilkS")
+		(layer "F.SilkS" knockout)
 		(effects
 			(font
@@
 	(gr_text "MOD"
 		(at 170.25 83.25 0)
-		(layer "F.SilkS")
+		(layer "F.SilkS" knockout)
 		(effects
 			(font
@@
 	(gr_text "PWR"
 		(at 170.25 85 0)
-		(layer "F.SilkS")
+		(layer "F.SilkS" knockout)
 		(effects
 			(font
@@
 	(gr_text "CN105"
 		(at 169.1 93.25 0)
-		(layer "F.SilkS")
+		(layer "F.SilkS" knockout)
 		(effects
 			(font
@@
 		)
 	)
+	(gr_text "ID"
+		(at 139.75 117.5 0)
+		(layer "F.SilkS" knockout)
+		(effects
+			(font
+				(size 1.2 1.5)
+				(thickness 0.18)
+			)
+			(justify left bottom)
+		)
+	)
 	(gr_text "GND"
 		(at 153.5 83.5 0)
@@
 	)
 	(gr_text "A"
-		(at 173 91.975 0)
+		(at 138.025 101.7625 270)
 		(layer "B.SilkS")
 		(effects
@@
 	)
 	(gr_text "SN"
-		(at 152.2375 115.5 0)
-		(layer "B.SilkS")
+		(at 132.25 106.5 270)
+		(layer "B.SilkS" knockout)
 		(effects
 			(font
@@
 	)
 	(gr_text "REV"
-		(at 178 92 0)
-		(layer "B.SilkS")
+		(at 138 106.7625 270)
+		(layer "B.SilkS" knockout)
 		(effects
 			(font
@@
 		)
 	)
-	(gr_text "MITSUBISHI\nCN105 CONTROLLER"
-		(at 151.1 103 0)
+	(gr_text "MITSUBISHI\nCN105 INTERFACE MODULE"
+		(at 181 96 0)
 		(layer "B.SilkS")
 		(effects
@@
 	)
 	(via
+		(at 184 99)
+		(size 0.8)
+		(drill 0.3)
+		(layers "F.Cu" "B.Cu")
+		(net 1)
+	)
+	(via
 		(at 153.1 94.9)
 		(size 0.8)
@@
 		(polygon
 			(pts
-				(xy 183 89) (xy 183 99.5) (xy 185 99.5) (xy 185 89)
+				(xy 183 89) (xy 183 98.5) (xy 185 98.5) (xy 185 89)
 			)
 		)

Commit message: hw: revA for fab
Parts:
- moved TP1 1.00 mm to (121.0, 98.0)
- moved TP3 1.00 mm to (121.0, 92.0)
Routing:
- net GND: track 46.5 -> 53.0 mm, vias 152 -> 160
- net /MODULE_SDA: track 36.4 -> 40.9 mm
- net /MODULE_SCL: track 35.8 -> 40.3 mm
- net /CN105_TX_IN_3V3: track 16.5 -> 21.0 mm
- net /CN105_RX_OUT_3V3: track 23.6 -> 28.1 mm
- net /CN105_OE: track 53.1 -> 48.6 mm
- net 5V_MODULE: track 20.2 -> 18.2 mm
- net /STATUS_LED: track 36.8 -> 35.2 mm
- added copper zone on F.Cu, net 5V_MODULE
