File: hw/Carrier_Board/Carrier_Board.kicad_sch (KiCad schematic)
At the start: 20 parts, among them J1 Conn_01x05

Commit message: hw: initial schematic mostly done, pushing for reference
Parts:
- removed C1, C2, C3, C4: C_Small, symbol Device:C_Small
- added C12, C14, C15, C16, C18, C7, C8, C9: 0.1u, Capacitor_SMD:C_0603_1608Metric_Pad1.08x0.95mm_HandSolder, symbol Device:C_Small
- added C13, C17: 4.7u, Capacitor_SMD:C_0805_2012Metric_Pad1.18x1.45mm_HandSolder, symbol Device:C_Small
- added D3, D4, D5: LED_Small_Filled, LED_SMD:LED_0603_1608Metric_Pad1.05x0.95mm_HandSolder, symbol Device:LED_Small_Filled
- added R1: 10K, Resistor_SMD:R_0603_1608Metric_Pad0.98x0.95mm_HandSolder, symbol Device:R_Small_US
- added R2, R3: 590, Resistor_SMD:R_0603_1608Metric_Pad0.98x0.95mm_HandSolder, symbol Device:R_Small_US
- added R4, R7: 270, Resistor_SMD:R_0603_1608Metric_Pad0.98x0.95mm_HandSolder, symbol Device:R_Small_US
- added R5, R6: 4.7K, Resistor_SMD:R_0603_1608Metric_Pad0.98x0.95mm_HandSolder, symbol Device:R_Small_US
- added U4: HDC1080, Package_SON:Texas_PWSON-N6, symbol Sensor_Humidity:HDC1080
- D1: renamed from D2; footprint (none) -> LED_SMD:LED_0603_1608Metric_Pad1.05x0.95mm_HandSolder; Comment (none) -> Green SMT LED
- F1: value Polyfuse_Small -> 500 mA; footprint (none) -> Fuse:Fuse_1206_3216Metric_Pad1.42x1.75mm_HandSolder; ManufacturerPartNumber (none) -> 0ZCJ0050AF2E
- TP1: renamed from TP5; footprint (none) -> TestPoint:TestPoint_Keystone_5005-5009_Compact
- TP2: renamed from TP6; footprint (none) -> TestPoint:TestPoint_Keystone_5005-5009_Compact
- TP3, TP4, TP7, TP8, TP9: footprint (none) -> TestPoint:TestPoint_Keystone_5005-5009_Compact
- TP5: renamed from TP1; footprint (none) -> TestPoint:TestPoint_Keystone_5005-5009_Compact
- TP6: renamed from TP2; footprint (none) -> TestPoint:TestPoint_Keystone_5005-5009_Compact
- renumbered D1 to D2
Connections:
- net 3V3: now also U2.1 (VCCA), U3.6 (VCCB), C12.2, C16.2, C17.2, C18.1, C9.2, D5.2 (A), R5.1, R6.1, U4.5 (VCC)
- net 5V_CN105: now also F1.1, U2.6 (VCCB), U3.1 (VCCA), C7.2, C8.2, D3.2 (A); no longer J1.3 (Pin_3)
- net 5V_MODULE: now also D1.2 (A), C13.2, C15.2
- net CN105_OE: now also U2.5 (OE), U3.5 (OE), R1.1
- net CN105_RX_OUT: now also U2.4 (BY)
- net CN105_RX_OUT_3V3: now also U2.3 (A)
- net CN105_TX_IN: now also U3.3 (A)
- net CN105_TX_IN_3V3: now also U3.4 (BY)
- net GND: now also U3.2 (GND), C12.1, C13.1, C14.1, C15.1, C16.1, C17.1, C18.2, C7.1, C8.1, C9.1, R1.2, R2.2, R3.2, R4.2, R7.2, U4.2 (GND)
- net CN105_5V_IN: now reaches F1.2
- net CN105_5V_IN: now also J1.3 (Pin_3), C14.2
- net at D1.1 (K): now also R2.1
- net STATUS_LED: now reaches U1.2 (GPIO5)
- net STATUS_LED: now also D4.2 (A)
- net MODULE_SDA: now reaches U1.8 (GPIO38)
- net MODULE_SDA: now also R6.2, U4.1 (SDA)
- net MODULE_SCL: now reaches U1.9 (GPIO39)
- net MODULE_SCL: now also R5.2, U4.6 (SCL)
- new net: D5.1 (K), R7.1
- new net: D3.1 (K), R3.1
- new net: D4.1 (K), R4.1
Other:
- note added: "CN105 INTERFACE"
- note added: "ESP32 MODULE"
- note added: "LEVEL SHIFTER"
- note added: "TEMP / HUMIDITY SENSOR"
- title: (none) -> CN105 Interface Board
- moved on the sheet: D1, D2, F1, J1, TP1, TP2, TP3, TP4, TP5, TP6, TP7, TP8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

Commit message: hw: initial layout done as well
Parts:
- removed C16: 0.1u, Capacitor_SMD:C_0603_1608Metric_Pad1.08x0.95mm_HandSolder, symbol Device:C_Small
- added R8, R9: 10K, Resistor_SMD:R_0603_1608Metric_Pad0.98x0.95mm_HandSolder, symbol Device:R_Small_US
- added TP1, TP2, TP3, TP4, TP5, TP6, TP7: TestPoint, TestPoint:TestPoint_Keystone_5000-5004_Miniature, symbol Connector:TestPoint
- J1: footprint (none) -> Carrier_Board:JST_PA_S05B
- TP10: renamed from TP3; footprint TestPoint:TestPoint_Keystone_5005-5009_Compact -> TestPoint:TestPoint_Keystone_5000-5004_Miniature
- TP11: renamed from TP4; footprint TestPoint:TestPoint_Keystone_5005-5009_Compact -> TestPoint:TestPoint_Keystone_5000-5004_Miniature
- TP12: renamed from TP5; footprint TestPoint:TestPoint_Keystone_5005-5009_Compact -> TestPoint:TestPoint_Keystone_5000-5004_Miniature
- TP13: renamed from TP6; footprint TestPoint:TestPoint_Keystone_5005-5009_Compact -> TestPoint:TestPoint_Keystone_5000-5004_Miniature
- TP14: renamed from TP7; footprint TestPoint:TestPoint_Keystone_5005-5009_Compact -> TestPoint:TestPoint_Keystone_5000-5004_Miniature
- TP15: renamed from TP8; footprint TestPoint:TestPoint_Keystone_5005-5009_Compact -> TestPoint:TestPoint_Keystone_5000-5004_Miniature
- TP16: renamed from TP9; footprint TestPoint:TestPoint_Keystone_5005-5009_Compact -> TestPoint:TestPoint_Keystone_5000-5004_Miniature
- TP8: renamed from TP1; footprint TestPoint:TestPoint_Keystone_5005-5009_Compact -> TestPoint:TestPoint_Keystone_5000-5004_Miniature
- TP9: renamed from TP2; footprint TestPoint:TestPoint_Keystone_5005-5009_Compact -> TestPoint:TestPoint_Keystone_5000-5004_Miniature
- U1: footprint (none) -> Carrier_Board:Atom_S3-Lite
- U3: renamed from U2; footprint (none) -> Package_TO_SOT_SMD:SOT-23-6_Handsoldering
- U4: renamed from U3; footprint (none) -> Package_TO_SOT_SMD:SOT-23-6_Handsoldering
- renumbered C18 to C1, C17 to C2, C15 to C3, C13 to C4, C14 to C5, C12 to C6, C9 to C7, C7 to C9, D5 to D1, D4 to D2, D1 to D3, D3 to D4, D2 to D5, R7 to R1, R4 to R2, R2 to R3, R5 to R4, R6 to R5, R3 to R6, R1 to R7, U4 to U2
Connections:
- net 3V3: now also TP4.1
- net 5V_CN105: now also R8.1, R9.1
- net CN105_RX_OUT: now also R9.2
- net CN105_RX_OUT_3V3: now also U1.9 (GPIO39); no longer U1.5 (GPIO8)
- net CN105_TX_IN: now also R8.2
- net CN105_TX_IN_3V3: now also U1.8 (GPIO38); no longer U1.4 (GPIO7)
- net GND: now also TP2.1, TP3.1, TP5.1
- net MODULE_SCL: now also U1.4 (GPIO7), TP6.1; no longer U1.9 (GPIO39)
- net MODULE_SDA: now also U1.5 (GPIO8), TP7.1; no longer U1.8 (GPIO38)
- net STATUS_LED: now also TP1.1
Other:
- moved on the sheet: D1, R1, R4, R5

Commit message: hw: ready for initial quoting
Parts:
- added C5: 4.7u, Capacitor_SMD:C_0805_2012Metric_Pad1.18x1.45mm_HandSolder, symbol Device:C_Small
- C1, C3: ManufacturerPartNumber (none) -> C0603C104K5RAC7411
- C10: renamed from C9; ManufacturerPartNumber (none) -> C0603C104K5RAC7411
- C2, C4: ManufacturerPartNumber (none) -> GRM21BR71C475KE51L; Voltage 25V -> 16V
- C6: renamed from C5; ManufacturerPartNumber (none) -> C0603C104K5RAC7411
- C7: renamed from C6; ManufacturerPartNumber (none) -> C0603C104K5RAC7411
- C8: renamed from C7; ManufacturerPartNumber (none) -> C0603C104K5RAC7411
- C9: renamed from C8; ManufacturerPartNumber (none) -> C0603C104K5RAC7411
- D1, D3, D4: ManufacturerPartNumber (none) -> LTST-C190GKT
- D2: ManufacturerPartNumber (none) -> LTST-C190AKT
- D5: ManufacturerPartNumber (none) -> SS12
- J1: value Conn_01x05 -> JST PA-Series Header (Right-Angle); ManufacturerPartNumber (none) -> S05B-PASK-2
- R1, R2: ManufacturerPartNumber (none) -> ERJ-3GEYJ271V
- R3, R6: value 590 -> 620; ManufacturerPartNumber (none) -> ERJ-3GEYJ621V
- R4, R5: ManufacturerPartNumber (none) -> ERJ-3GEYJ472V
- R7, R8, R9: ManufacturerPartNumber (none) -> ERJ-3GEYJ103V
- U3: value ~ -> (none)
Connections:
- net 5V_CN105: now also C5.2
- net GND: now also C5.1
Other:
- moved on the sheet: C10, C2, C3, C7, C8, C9, D3, D5, R3, R7, R8, R9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

Commit message: hw: revA for fab
Parts:
- U3: value (none) -> ~
Changed lines of the file:
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@@
 			)
 		)
-		(property "Value" ""
+		(property "Value" "~"
 			(at 212.09 144.78 0)
 			(effects
